Commit message: update hardware mecanum wheel system

File: linorobot2_description/urdf/controllers/mecanum_ros2_control.urdf.xacro (robot description, xacro)
@@ -1,6 +1,6 @@
 <?xml version="1.0"?>
 <robot xmlns:xacro="http://www.ros.org/wiki/xacro">
-    <xacro:macro name="insert_ros2_control_mecanum" params="prefix is_sim:=^|false robot_port_name robot_baudrate">
-        <ros2_control name="${prefix}minibot_system" type="system">
+    <xacro:macro name="insert_ros2_control_mecanum" params="is_sim:=^|false robot_port_name robot_baudrate">
+        <ros2_control name="$minibot_system" type="system">
             <xacro:if value="$(arg is_sim)">
                 <hardware>
@@ -15,37 +15,4 @@
                 </hardware>
             </xacro:unless>
-            <!-- 20230614 update macanumwheel_system-->
-            <joint name="${prefix}front_l_wheel_joint">
-                <command_interface name="velocity">
-                    <param name="min">-1.0</param>
-                    <param name="max">1.0</param>
-                </command_interface>
-                <state_interface name="position"/>
-                <state_interface name="velocity"/>
-            </joint>
-            <joint name="${prefix}front_r_wheel_joint">
-                <command_interface name="velocity">
-                    <param name="min">-1.0</param>
-                    <param name="max">1.0</param>
-                </command_interface>
-                <state_interface name="position"/>
-                <state_interface name="velocity"/>
-            </joint>
-            <joint name="${prefix}rear_l_wheel_joint">
-                <command_interface name="velocity">
-                    <param name="min">-1.0</param>
-                    <param name="max">1.0</param>
-                </command_interface>
-                <state_interface name="position"/>
-                <state_interface name="velocity"/>
-            </joint>
-            <joint name="${prefix}rear_r_wheel_joint">
-                <command_interface name="velocity">
-                    <param name="min">-1.0</param>
-                    <param name="max">1.0</param>
-                </command_interface>
-                <state_interface name="position"/>
-                <state_interface name="velocity"/>
-            </joint>
             <gpio name="gpio">
                 <!-- <command_interface name="set_enable_motor"/> -->

File: linorobot2_description/urdf/mech/mecanum_wheel.urdf.xacro (robot description, xacro)
@@ -2,4 +2,6 @@
 <robot xmlns:xacro="http://ros.org/wiki/xacro">
   <xacro:macro name="mecanum_wheel" params="side radius width pos_x pos_y pos_z mass">
+    <!-- 20230615 update macanumwheel_system-->
+    <!--          port, baudrate update-->
     <link name="${side}_wheel_link">
       <visual>
@@ -45,4 +47,10 @@
       <child link="${side}_wheel_link"/>
       <origin xyz="${pos_x} ${pos_y} ${pos_z}" rpy="0 0 0"/>
+      <command_interface name="velocity">
+        <param name="min">-1.0</param>
+        <param name="max">1.0</param>
+      </command_interface>
+      <state_interface name="position"/>
+      <state_interface name="velocity"/>
     </joint>
   </xacro:macro>

File: linorobot2_description/urdf/robots/mecanum.urdf.xacro (robot description, xacro)
@@ -8,15 +8,14 @@
   <xacro:include filename="$(find linorobot2_description)/urdf/sensors/depth_sensor.urdf.xacro" />
   <xacro:include filename="$(find linorobot2_description)/urdf/controllers/omni_drive.urdf.xacro" />
-  <xacro:include filename="$(find linorobot2_description)/urdf/controllers/mecanum_ros2_control.urdf.xacro" />
-   <xacro:arg name="prefix" default=""/>
-   <xacro:arg name="is_sim" default="false"/>
-   <xacro:arg name="robot_port_name" default="/dev/ttySTM32"/>
-   <xacro:arg name="robot_baudrate" default="500000"/>
-   <xacro:property name="prefix" value="$(arg prefix)"/>
+  <xacro:include filename="$(find linorobot2_description)/urdf/controllers/mecanum_ros2_control.urdf.xacro"/>
+  <xacro:property name="is_sim" default="false"/>
+  <xacro:property name="robot_port_name" default="/dev/ttySTM32"/>
+  <xacro:property name="robot_baudrate" default="500000"/>
    <!-- insert robot base -->
-    <xacro:insert_ros2_control_mecanum prefix="$(arg prefix)" is_sim="$(arg is_sim)" robot_port_name="$(arg robot_port_name)" robot_baudrate="$(arg robot_baudrate)"/>
-    <xacro:if value="$(arg is_sim)">
+    <!-- <xacro:property name="prefix" value=""/> -->
+    <xacro:insert_ros2_control_mecanum is_sim="$(arg is_sim)" robot_port_name="$(arg robot_port_name)" robot_baudrate="$(arg robot_baudrate)"/>
+    <!-- <xacro:if value="$(arg is_sim)">
         <xacro:insert_gazebo prefix="$(arg prefix)"/>
-    </xacro:if>
+    </xacro:if>  -->
   <xacro:base
     length="${base_length}"
@@ -70,4 +69,5 @@
     <xacro:insert_block name="depth_sensor_pose" />
   </xacro:depth_sensor>
+   <!-- <xacro:insert_ros2_control_mecanum prefix="$(arg prefix)" is_sim="$(arg is_sim)" robot_port_name="$(arg robot_port_name)" robot_baudrate="$(arg robot_baudrate)"/> -->
   <xacro:omni_drive_controller/>
 </robot>

Commit message: change xacro arg -> property)

File: linorobot2_description/urdf/controllers/mecanum_ros2_control.urdf.xacro (robot description, xacro)
@@ -1,6 +1,6 @@
 <?xml version="1.0"?>
 <robot xmlns:xacro="http://www.ros.org/wiki/xacro">
-    <xacro:macro name="insert_ros2_control" params="prefix is_sim:=^|false robot_port_name robot_baudrate">
-        <ros2_control name="${prefix}minibot_system" type="system">
+    <xacro:macro name="insert_ros2_control_mecanum" params="is_sim:=^|false robot_port_name robot_baudrate">
+        <ros2_control name="$minibot_system" type="system">
             <xacro:if value="$(arg is_sim)">
                 <hardware>
@@ -15,22 +15,6 @@
                 </hardware>
             </xacro:unless>
-            <joint name="${prefix}l_wheel_joint">
-                <command_interface name="velocity">
-                    <param name="min">-1.0</param>
-                    <param name="max">1.0</param>
-                </command_interface>
-                <state_interface name="position"/>
-                <state_interface name="velocity"/>
-            </joint>
-            <joint name="${prefix}r_wheel_joint">
-                <command_interface name="velocity">
-                    <param name="min">-1.0</param>
-                    <param name="max">1.0</param>
-                </command_interface>
-                <state_interface name="position"/>
-                <state_interface name="velocity"/>
-            </joint>
             <gpio name="gpio">
-                <command_interface name="set_enable_motor"/>
+                <!-- <command_interface name="set_enable_motor"/> -->
                 <state_interface name="motor_enabled"/>
                 <command_interface name="set_l_lamp_command"/>

File: linorobot2_description/urdf/robots/mecanum.urdf.xacro (robot description, xacro)
@@ -8,16 +8,11 @@
   <xacro:include filename="$(find linorobot2_description)/urdf/sensors/depth_sensor.urdf.xacro" />
   <xacro:include filename="$(find linorobot2_description)/urdf/controllers/omni_drive.urdf.xacro" />
-   <xacro:arg name="prefix" default=""/>
-   <xacro:arg name="is_sim" default="false"/>
-   <xacro:arg name="robot_port_name" default="/dev/ttySTM32"/>
-   <xacro:arg name="robot_baudrate" default="500000"/>
-   <xacro:property name="prefix" value="$(arg prefix)"/>
-  <!-- insert robot base
-    <xacro:insert_robot prefix="$(arg prefix)"/>
-    <xacro:insert_ros2_control prefix="$(arg prefix)" is_sim="$(arg is_sim)" robot_port_name="$(arg robot_port_name)" robot_baudrate="$(arg robot_baudrate)"/>
-  -->
+  <xacro:include filename="$(find linorobot2_description)/urdf/controllers/mecanum_ros2_control.urdf.xacro"/>
+   <!-- insert robot base -->
+    <!-- <xacro:property name="prefix" value=""/> -->
+    <xacro:insert_ros2_control_mecanum is_sim="${is_sim}" robot_port_name="${robot_port_name}" robot_baudrate="${robot_baudrate}"/>
     <!-- <xacro:if value="$(arg is_sim)">
-        <xacro:insert_gazebo prefix="$(arg prefix)"/> Only GAZEBO
-    </xacro:if> -->
+        <xacro:insert_gazebo prefix="$(arg prefix)"/>
+    </xacro:if>  -->
   <xacro:base
     length="${base_length}"
@@ -71,4 +66,5 @@
     <xacro:insert_block name="depth_sensor_pose" />
   </xacro:depth_sensor>
+   <!-- <xacro:insert_ros2_control_mecanum prefix="$(arg prefix)" is_sim="$(arg is_sim)" robot_port_name="$(arg robot_port_name)" robot_baudrate="$(arg robot_baudrate)"/> -->
   <xacro:omni_drive_controller/>
 </robot>

Commit message: change xacro arg -> property 5th

File: linorobot2_description/urdf/controllers/mecanum_ros2_control.urdf.xacro (robot description, xacro)
@@ -1,5 +1,5 @@
 <?xml version="1.0"?>
 <robot xmlns:xacro="http://www.ros.org/wiki/xacro">
-    <xacro:macro name="insert_ros2_control_mecanum" params="is_sim:=^|false robot_port_name robot_baudrate">
+    <xacro:macro name="insert_ros2_control_mecanum" params="is_sim robot_port_name robot_baudrate">
         <ros2_control name="$minibot_system" type="system">
             <xacro:if value="$(arg is_sim)">
@@ -11,6 +11,6 @@
                 <hardware>
                     <plugin>minibot_hardware/MinibotSystemHardware</plugin>
-                    <param name="port_name">$(arg robot_port_name)</param>
-                    <param name="baudrate">$(arg robot_baudrate)</param>
+                    <param name="port_name">${robot_port_name}</param>
+                    <param name="baudrate">${robot_baudrate}</param>
                 </hardware>
             </xacro:unless>

Commit message: change xacro property to arg

File: linorobot2_description/urdf/controllers/mecanum_ros2_control.urdf.xacro (robot description, xacro)
@@ -2,5 +2,5 @@
 <robot xmlns:xacro="http://www.ros.org/wiki/xacro">
     <xacro:macro name="insert_ros2_control_mecanum" params="is_sim robot_port_name robot_baudrate">
-        <ros2_control name="$minibot_system" type="system">
+        <ros2_control name="minibot_system" type="system">
             <xacro:if value="$(arg is_sim)">
                 <hardware>
@@ -11,6 +11,6 @@
                 <hardware>
                     <plugin>minibot_hardware/MinibotSystemHardware</plugin>
-                    <param name="port_name">${robot_port_name}</param>
-                    <param name="baudrate">${robot_baudrate}</param>
+                    <param name="port_name">$(arg robot_port_name)</param>
+                    <param name="baudrate">$(arg robot_baudrate)</param>
                 </hardware>
             </xacro:unless>

File: linorobot2_description/urdf/mecanum_properties.urdf.xacro (robot description, xacro)
@@ -13,6 +13,6 @@
   <xacro:property name="wheel_torque" value="20" />
   <xacro:property name="is_sim" value="false"/>
-  <!-- <xacro:property name="robot_port_name" value="/dev/ttySTM32"/> -->
-  <!-- <xacro:property name="robot_baudrate" value="500000"/> -->
+  <xacro:arg name="robot_port_name" default="/dev/ttySTM32"/>
+  <xacro:arg name="robot_baudrate" default="500000"/>
   <xacro:property name="laser_pose">
     <origin xyz="-0.0475 0 0.125" rpy="0 0 0"/>

File: linorobot2_description/urdf/robots/mecanum.urdf.xacro (robot description, xacro)
@@ -11,5 +11,5 @@
    <!-- insert robot base -->
     <!-- <xacro:property name="prefix" value=""/> -->
-    <xacro:insert_ros2_control_mecanum is_sim="false" robot_port_name="/dev/ttySTM32" robot_baudrate="500000"/>
+    <xacro:insert_ros2_control_mecanum is_sim="$(arg is_sim)" robot_port_name="$(arg robot_port_name)" robot_baudrate="$(arg robot_baudrate)"/>
     <!-- <xacro:if value="$(arg is_sim)">
         <xacro:insert_gazebo prefix="$(arg prefix)"/>
