Commit message: property update

File: linorobot2_description/urdf/mecanum_properties.urdf.xacro (robot description, xacro)
@@ -12,4 +12,7 @@
   <xacro:property name="wheel_mass" value=".6" />
   <xacro:property name="wheel_torque" value="20" />
+  <xacro:property name="is_sim" default="false"/>
+  <xacro:property name="robot_port_name" default="/dev/ttySTM32"/>
+  <xacro:property name="robot_baudrate" default="500000"/>
   <xacro:property name="laser_pose">
     <origin xyz="-0.0475 0 0.125" rpy="0 0 0"/>

File: linorobot2_description/urdf/robots/mecanum.urdf.xacro (robot description, xacro)
@@ -9,7 +9,4 @@
   <xacro:include filename="$(find linorobot2_description)/urdf/controllers/omni_drive.urdf.xacro" />
   <xacro:include filename="$(find linorobot2_description)/urdf/controllers/mecanum_ros2_control.urdf.xacro"/>
-  <xacro:property name="is_sim" default="false"/>
-  <xacro:property name="robot_port_name" default="/dev/ttySTM32"/>
-  <xacro:property name="robot_baudrate" default="500000"/>
    <!-- insert robot base -->
     <!-- <xacro:property name="prefix" value=""/> -->

Commit message: change xacro arg -> property 2nd

File: linorobot2_description/urdf/mecanum_properties.urdf.xacro (robot description, xacro)
@@ -12,7 +12,7 @@
   <xacro:property name="wheel_mass" value=".6" />
   <xacro:property name="wheel_torque" value="20" />
-  <xacro:property name="is_sim" default="false"/>
-  <xacro:property name="robot_port_name" default="/dev/ttySTM32"/>
-  <xacro:property name="robot_baudrate" default="500000"/>
+  <xacro:property name="is_sim" value="false"/>
+  <xacro:property name="robot_port_name" value="/dev/ttySTM32"/>
+  <xacro:property name="robot_baudrate" value="500000"/>
   <xacro:property name="laser_pose">
     <origin xyz="-0.0475 0 0.125" rpy="0 0 0"/>

Commit message: change xacro arg -> property 3rd

File: linorobot2_description/urdf/mecanum_properties.urdf.xacro (robot description, xacro)
@@ -13,6 +13,6 @@
   <xacro:property name="wheel_torque" value="20" />
   <xacro:property name="is_sim" value="false"/>
-  <xacro:property name="robot_port_name" value="/dev/ttySTM32"/>
-  <xacro:property name="robot_baudrate" value="500000"/>
+  <!-- <xacro:property name="robot_port_name" value="/dev/ttySTM32"/> -->
+  <!-- <xacro:property name="robot_baudrate" value="500000"/> -->
   <xacro:property name="laser_pose">
     <origin xyz="-0.0475 0 0.125" rpy="0 0 0"/>

File: linorobot2_description/urdf/robots/mecanum.urdf.xacro (robot description, xacro)
@@ -11,5 +11,5 @@
    <!-- insert robot base -->
     <!-- <xacro:property name="prefix" value=""/> -->
-    <xacro:insert_ros2_control_mecanum is_sim="${is_sim}" robot_port_name="${robot_port_name}" robot_baudrate="${robot_baudrate}"/>
+    <xacro:insert_ros2_control_mecanum is_sim="false" robot_port_name="/dev/ttySTM32" robot_baudrate="500000"/>
     <!-- <xacro:if value="$(arg is_sim)">
         <xacro:insert_gazebo prefix="$(arg prefix)"/>

Commit message: tmp

File: linorobot2_description/urdf/mecanum_properties.urdf.xacro (robot description, xacro)
@@ -12,7 +12,7 @@
   <xacro:property name="wheel_mass" value=".6" />
   <xacro:property name="wheel_torque" value="20" />
-  <xacro:property name="is_sim" value="false"/>
-  <!-- <xacro:property name="robot_port_name" value="/dev/ttySTM32"/> -->
-  <!-- <xacro:property name="robot_baudrate" value="500000"/> -->
+  <xacro:arg name="is_sim" default="false"/>
+  <xacro:arg name="robot_port_name" default="/dev/ttySTM32"/>
+  <xacro:arg name="robot_baudrate" default="500000"/>
   <xacro:property name="laser_pose">
     <origin xyz="-0.0475 0 0.125" rpy="0 0 0"/>
