Commit message: xacro file fixed

File: linorobot2_description/urdf/robots/mecanum.urdf.xacro (robot description, xacro)
@@ -8,4 +8,16 @@
   <xacro:include filename="$(find linorobot2_description)/urdf/sensors/depth_sensor.urdf.xacro" />
   <xacro:include filename="$(find linorobot2_description)/urdf/controllers/omni_drive.urdf.xacro" />
+   <xacro:arg name="prefix" default=""/>
+   <xacro:arg name="is_sim" default="false"/>
+   <xacro:arg name="robot_port_name" default="/dev/ttySTM32"/>
+   <xacro:arg name="robot_baudrate" default="500000"/>
+   <xacro:property name="prefix" value="$(arg prefix)"/>
+  <!-- insert robot base
+    <xacro:insert_robot prefix="$(arg prefix)"/>
+    <xacro:insert_ros2_control prefix="$(arg prefix)" is_sim="$(arg is_sim)" robot_port_name="$(arg robot_port_name)" robot_baudrate="$(arg robot_baudrate)"/>
+  -->
+    <!-- <xacro:if value="$(arg is_sim)">
+        <xacro:insert_gazebo prefix="$(arg prefix)"/> Only GAZEBO
+    </xacro:if> -->
   <xacro:base
     length="${base_length}"

File: linorobot2_description/urdf/sensors/depth_sensor.urdf.xacro (robot description, xacro)
@@ -4,5 +4,5 @@
     <link name="camera_link">
       <visual>
-        <origin xyz="0 0 0" rpy="0 0 0"/>
+        <origin xyz="-0.02 0 0.02" rpy="0 0 0"/>
         <geometry>
           <box size="0.030 0.124 0.030"/>

File: linorobot2_description/urdf/sensors/laser.urdf.xacro (robot description, xacro)
@@ -4,7 +4,7 @@
     <link name="${frame_id}">
       <visual>
-        <origin xyz="0 0 -0.025" rpy="0 0 0"/>
+        <origin xyz="0.16 0 -0.05" rpy="0 0 0"/>
         <geometry>
-          <cylinder radius="0.0375" length="0.05"/>
+            <mesh filename="package://minibot_description/meshes/visual/ydlidar_x2_assy.dae" scale="1 1 1"/>
         </geometry>
         <material name="green">
@@ -13,12 +13,13 @@
       </visual>
       <collision>
-        <origin xyz="0 0 -0.025" rpy="0 0 0"/>
+        <origin xyz="0.16 0 -0.05" rpy="0 0 0"/>
         <geometry>
+          <mesh filename="package://minibot_description/meshes/collision/ydlidar_x2_assy.stl" scale="1 1 1"/>
           <cylinder radius="0.0375" length="0.05"/>
         </geometry>
       </collision>
       <inertial>
-        <origin xyz="0 0 0" rpy="0 0 0"/>
-        <mass value="0.1"/>
+        <origin xyz="0.007 0 0.025" rpy="0 0 0"/>
+        <mass value="0.150"/>
         <inertia ixx="${(2/5) * 0.1 * (0.0375 * 0.0375)}" ixy="0" ixz="0"
                  iyy="${(2/5) * 0.1 * (0.0375 * 0.0375)}" iyz="0"

Commit message: hardware interface fixed

File: linorobot2_description/urdf/robots/mecanum.urdf.xacro (robot description, xacro)
@@ -8,4 +8,5 @@
   <xacro:include filename="$(find linorobot2_description)/urdf/sensors/depth_sensor.urdf.xacro" />
   <xacro:include filename="$(find linorobot2_description)/urdf/controllers/omni_drive.urdf.xacro" />
+  <xacro:include filename="$(find linorobot2_description)/urdf/controllers/mecanum_ros2_control.urdf.xacro" />
    <xacro:arg name="prefix" default=""/>
    <xacro:arg name="is_sim" default="false"/>
@@ -13,11 +14,10 @@
    <xacro:arg name="robot_baudrate" default="500000"/>
    <xacro:property name="prefix" value="$(arg prefix)"/>
-  <!-- insert robot base
+   <!-- insert robot base -->
     <xacro:insert_robot prefix="$(arg prefix)"/>
-    <xacro:insert_ros2_control prefix="$(arg prefix)" is_sim="$(arg is_sim)" robot_port_name="$(arg robot_port_name)" robot_baudrate="$(arg robot_baudrate)"/>
-  -->
-    <!-- <xacro:if value="$(arg is_sim)">
-        <xacro:insert_gazebo prefix="$(arg prefix)"/> Only GAZEBO
-    </xacro:if> -->
+    <xacro:insert_ros2_control_mecanum prefix="$(arg prefix)" is_sim="$(arg is_sim)" robot_port_name="$(arg robot_port_name)" robot_baudrate="$(arg robot_baudrate)"/>
+    <xacro:if value="$(arg is_sim)">
+        <xacro:insert_gazebo prefix="$(arg prefix)"/>
+    </xacro:if>
   <xacro:base
     length="${base_length}"

File: linorobot2_description/urdf/sensors/laser.urdf.xacro (robot description, xacro)
@@ -4,7 +4,7 @@
     <link name="${frame_id}">
       <visual>
-        <origin xyz="0.16 0 -0.05" rpy="0 0 0"/>
+        <origin xyz="0.16 0 0.02" rpy="0 0 0"/>
         <geometry>
-            <mesh filename="package://minibot_description/meshes/visual/ydlidar_x2_assy.dae" scale="1 1 1"/>
+          <cylinder radius="0.0375" length="0.05"/>
         </geometry>
         <material name="green">
@@ -13,7 +13,6 @@
       </visual>
       <collision>
-        <origin xyz="0.16 0 -0.05" rpy="0 0 0"/>
+        <origin xyz="0.16 0 0.02" rpy="0 0 0"/>
         <geometry>
-          <mesh filename="package://minibot_description/meshes/collision/ydlidar_x2_assy.stl" scale="1 1 1"/>
           <cylinder radius="0.0375" length="0.05"/>
         </geometry>

Commit message: add system

File: linorobot2_description/urdf/robots/mecanum.urdf.xacro (robot description, xacro)
@@ -5,14 +5,7 @@
   <xacro:include filename="$(find linorobot2_description)/urdf/mech/mecanum_wheel.urdf.xacro" />
   <xacro:include filename="$(find linorobot2_description)/urdf/sensors/imu.urdf.xacro" />
-  <xacro:include filename="$(find linorobot2_description)/urdf/sensors/generic_laser.urdf.xacro" />
+  <!-- <xacro:include filename="$(find linorobot2_description)/urdf/sensors/generic_laser.urdf.xacro" /> -->
   <xacro:include filename="$(find linorobot2_description)/urdf/sensors/depth_sensor.urdf.xacro" />
   <xacro:include filename="$(find linorobot2_description)/urdf/controllers/omni_drive.urdf.xacro" />
-  <xacro:include filename="$(find linorobot2_description)/urdf/controllers/mecanum_ros2_control.urdf.xacro"/>
-   <!-- insert robot base -->
-    <!-- <xacro:property name="prefix" value=""/> -->
-    <xacro:insert_ros2_control_mecanum is_sim="false" robot_port_name="/dev/ttySTM32" robot_baudrate="500000"/>
-    <!-- <xacro:if value="$(arg is_sim)">
-        <xacro:insert_gazebo prefix="$(arg prefix)"/>
-    </xacro:if>  -->
   <xacro:base
     length="${base_length}"
@@ -24,5 +17,5 @@
 />
   <xacro:mecanum_wheel
-    side="front_left"
+    side="fl"
     radius="${wheel_radius}"
     width="${wheel_width}"
@@ -33,5 +26,5 @@
   />
   <xacro:mecanum_wheel
-    side="front_right"
+    side="fr"
     radius="${wheel_radius}"
     width="${wheel_width}"
@@ -42,5 +35,5 @@
   />
   <xacro:mecanum_wheel
-    side="rear_left"
+    side="rl"
     radius="${wheel_radius}"
     width="${wheel_width}"
@@ -51,5 +44,5 @@
   />
   <xacro:mecanum_wheel
-    side="rear_right"
+    side="rr"
     radius="${wheel_radius}"
     width="${wheel_width}"
@@ -66,4 +59,22 @@
     <xacro:insert_block name="depth_sensor_pose" />
   </xacro:depth_sensor>
+  <ros2_control name="secser_system" type="system">
+    <xacro:unless value="$(arg is_sim)">
+        <hardware>
+            <plugin>minibot_hardware/MinibotSystemHardware</plugin>
+            <param name="port_name">/dev/ttySTM32</param>
+            <param name="baudrate">1000000</param>
+        </hardware>
+    </xacro:unless>
+    <gpio name="gpio">
+        <!-- <command_interface name="set_enable_motor"/> -->
+        <state_interface name="motor_enabled"/>
+        <command_interface name="set_l_lamp_command"/>
+        <command_interface name="set_r_lamp_command"/>
+        <state_interface name="l_lamp_state"/>
+        <state_interface name="r_lamp_state"/>
+        <state_interface name="range_sensor_state"/>
+    </gpio>
+</ros2_control>
    <!-- <xacro:insert_ros2_control_mecanum prefix="$(arg prefix)" is_sim="$(arg is_sim)" robot_port_name="$(arg robot_port_name)" robot_baudrate="$(arg robot_baudrate)"/> -->
   <xacro:omni_drive_controller/>
