Commit message: complete description

File: minibot_description/urdf/minibot.urdf.xacro (robot description, xacro)
@@ -1,124 +1,95 @@
 <?xml version="1.0"?>
 <robot xmlns:xacro="http://www.ros.org/wiki/xacro">
-    <xacro:macro name="insert_robot" params="prefix">
-        <xacro:property name="wheel_diameter" value="0.068"/>
-        <xacro:property name="wheel_speration" value="0.180"/>
+    <xacro:macro name="insert_robot" params="prefix length width height mass wheel_radius wheel_pos_z">
         <link name="${prefix}base_footprint"/>
         <link name="${prefix}base_link">
-            <visual>
-                <origin xyz="0 0 0" rpy="0 0 0"/>
-                <geometry>
-                    <mesh filename="package://minibot_description/meshes/visual/base_link.dae" scale="1 1 1"/>
-                </geometry>
-            </visual>
+          <visual>
+              <origin xyz="0 0 0" rpy="0 0 0"/>
+              <geometry>
+                <box size="${length} ${width} ${height}"/>
+                <!-- <mesh filename="" scale="0.001 0.001 0.001"/> -->
+              </geometry>
+                <material name="yellow">
+                <color rgba="0.8784 0.6627 0.6627 1.0"/>
+                </material>
+         </visual>
             <collision>
                 <origin xyz="0 0 0" rpy="0 0 0"/>
                 <geometry>
-                    <mesh filename="package://minibot_description/meshes/collision/base_link.stl" scale="1 1 1"/>
+                    <box size="${length} ${width} ${height}"/>
                 </geometry>
             </collision>
-            <inertial>
-                <origin xyz="-0.02 0 0.028" rpy="0 0 0"/>
-                <mass value="2.0"/>
-                <!-- <inertia ixx="0.000213" ixy="0" ixz="0" iyy="0.007034" iyz="0" izz="0.008104"/> -->
-                <inertia ixx="0.01" ixy="0" ixz="0" iyy="0.01" iyz="0" izz="0.01"/>
-            </inertial>
+              <inertial>
+                <origin xyz="0 0 0" rpy="0 0 0"/>
+              <mass value="${mass}"/>
+              <inertia ixx="${(1/12) * mass * ((width  * width)  + (height * height))}" ixy="0.0" ixz="0.0"
+                    iyy="${(1/12) * mass * ((length * length) + (height * height))}" iyz="0.0"
+                    izz="${(1/12) * mass * ((length * length) + (width  * width))}"/>
+              </inertial>
         </link>
-        <joint name="${prefix}base_link_fixed_joint" type="fixed">
-            <parent link="${prefix}base_footprint"/>
-            <child link="${prefix}base_link"/>
-            <origin xyz="0 0 ${wheel_diameter/2}" rpy="0 0 0"/>
-        </joint>
-        <xacro:macro name="insert_wheel" params="parent prefix prefix_dir dir">
-            <link name="${prefix}${prefix_dir}_wheel">
+         <gazebo reference="base_link">
+            <visual>
+                <material>
+                    <ambient>0.8392 0.6314 0.0 1.0</ambient>
+                    <diffuse>0.8392 0.6314 0.0 1.0</diffuse>
+                    <specular>0.99 0.99 0.99 1.0</specular>
+                    <emissive>0.0 0.0 0.0 0.0</emissive>
+                </material>
+            </visual>
+        </gazebo>
+        <joint name="base_to_footprint" type="fixed">
+        <parent link="base_footprint"/>
+        <child link="base_link"/>
+        <origin xyz="0 0 ${wheel_radius - wheel_pos_z}" rpy="0 0 0"/>
+      </joint>
+     </xacro:macro>
+     <xacro:macro name="mecanum_wheel" params="side radius width pos_x pos_y pos_z mass">
+            <link name="${side}_wheel_link">
                 <visual>
-                    <origin xyz="0 0 0" rpy="0 0 ${dir * pi/2}"/>
+                    <origin xyz="0 0 0" rpy="${pi/2} 0 0"/>
                     <geometry>
-                        <mesh filename="package://minibot_description/meshes/visual/wheel.dae" scale="1 1 1"/>
+                        <cylinder radius="${radius}" length="${width}"/>
                     </geometry>
+                    <material name="blue">
+                        <color rgba="0.1764 0.4588 0.8509 1.0"/>
+                    </material>
                 </visual>
-                <collision>
-                    <origin xyz="0 0 0" rpy="0 0 ${dir * pi/2}"/>
-                    <geometry>
-                        <mesh filename="package://minibot_description/meshes/collision/wheel.stl" scale="1 1 1"/>
-                    </geometry>
-                </collision>
-                <inertial>
-                    <origin xyz="0 0 0" rpy="0 0 0"/>
-                    <mass value="0.200"/>
-                    <!-- <inertia ixx="0.000067" ixy="0" ixz="0" iyy="0.000113" iyz="0" izz="0.000067"/> -->
-                    <!-- For stable on GAZEBO. Force Inertial value to LARGE value -->
-                    <inertia ixx="0.1" ixy="0" ixz="0" iyy="0.1" iyz="0" izz="0.1"/>
-                </inertial>
-            </link>
-            <joint name="${prefix}${prefix_dir}_wheel_joint" type="continuous">
-                <parent link="${parent}"/>
-                <child link="${prefix}${prefix_dir}_wheel"/>
-                <axis xyz="0 1 0"/>
-                <origin xyz="0 ${dir * wheel_speration/2} 0" rpy="0 0 0"/>
-            </joint>
-        </xacro:macro>
-        <xacro:insert_wheel parent="${prefix}base_link" prefix="${prefix}" prefix_dir="l" dir="1" />
-        <xacro:insert_wheel parent="${prefix}base_link" prefix="${prefix}" prefix_dir="r" dir="-1" />
-        <link name="${prefix}front_camera_mount">
-            <visual>
-                <origin xyz="0 0 0" rpy="0 0 0"/>
-                <geometry>
-                    <mesh filename="package://minibot_description/meshes/visual/front_camera.dae" scale="1 1 1"/>
-                </geometry>
-            </visual>
-            <collision>
-                <origin xyz="0 0 0" rpy="0 0 0"/>
-                <geometry>
-                    <mesh filename="package://minibot_description/meshes/collision/front_camera.stl" scale="1 1 1"/>
-                </geometry>
-            </collision>
-            <inertial>
-                <origin xyz="0.005 0 0.013" rpy="0 0 0"/>
-                <mass value="0.050000"/>
-                <inertia ixx="0.000005" ixy="0" ixz="-0.000001" iyy="0.000004" iyz="0" izz="0.000003"/>
-            </inertial>
-        </link>
-        <joint name="${prefix}front_camera_mount_fixed_joint" type="fixed">
-            <parent link="${prefix}base_link"/>
-            <child link="${prefix}front_camera_mount"/>
-            <origin xyz="0.045 0 0.085" rpy="0 0 0"/>
-        </joint>
-        <link name="${prefix}camera_link"/>
-        <joint name="${prefix}camera_link_fixed_joint" type="fixed">
-            <parent link="${prefix}front_camera_mount"/>
-            <child link="${prefix}camera_link"/>
-            <origin xyz="0.0111 0 0.0193" rpy="0 ${pi/2} 0"/>
-        </joint>
-        <link name="${prefix}ul_sensor_mount">
-            <visual>
-                <origin xyz="0 0 0" rpy="0 0 0"/>
-                <geometry>
-                    <mesh filename="package://minibot_description/meshes/visual/ul_sensor.dae" scale="1 1 1"/>
-                </geometry>
-            </visual>
-            <collision>
-                <origin xyz="0 0 0" rpy="0 0 0"/>
-                <geometry>
-                    <mesh filename="package://minibot_description/meshes/collision/ul_sensor.stl" scale="1 1 1"/>
-                </geometry>
-            </collision>
-            <inertial>
-                <origin xyz="0.005 0 0.013" rpy="0 0 0"/>
-                <mass value="0.050000"/>
-                <inertia ixx="0.000005" ixy="0" ixz="-0.000001" iyy="0.000004" iyz="0" izz="0.000003"/>
-            </inertial>
-        </link>
-        <joint name="${prefix}ul_sensor_mount_fixed_joint" type="fixed">
-            <parent link="${prefix}base_link"/>
-            <child link="${prefix}ul_sensor_mount"/>
-            <origin xyz="0.03 0 0.01" rpy="0 0 0"/>
-        </joint>
-        <link name="${prefix}ul_sensor_link"/>
-        <joint name="${prefix}ul_sensor_link_fixed_joint" type="fixed">
-            <parent link="${prefix}ul_sensor_mount"/>
-            <child link="${prefix}ul_sensor_link"/>
-            <origin xyz="0.02 0 0" rpy="0 0 0"/>
-        </joint>
+      <collision>
+        <origin xyz="0 0 0" rpy="${pi/2} 0 0"/>
+        <geometry>
+          <cylinder radius="${radius}" length="${width}"/>
+        </geometry>
+      </collision>
+      <inertial>
+        <origin xyz="0 0 0" rpy="0 0 0"/>
+        <mass value="${mass}"/>
+        <inertia ixx="${(2/5) * mass * (radius * radius)}" ixy="0" ixz="0"
+                 iyy="${(2/5) * mass * (radius * radius)}" iyz="0"
+                 izz="${(2/5) * mass * (radius * radius)}" />
+      </inertial>
+    </link>
+    <gazebo reference="${side}_wheel_link">
+        <mu1>0.01</mu1>
+        <mu2>0.01</mu2>
+    </gazebo>
+    <gazebo reference="${side}_wheel_link">
+      <visual>
+        <material>
+          <ambient>0.1764 0.4588 0.8509 1.0</ambient>
+          <diffuse>0.1764 0.4588 0.8509 1.0</diffuse>
+          <specular>0.1764 0.4588 0.8509 1.0</specular>
+          <emissive>0.0 0.0 0.0 0.0</emissive>
+        </material>
+      </visual>
+    </gazebo>
+    <joint name="${side}_wheel_joint" type="continuous">
+      <axis xyz="0 1 0" />
+      <parent link="base_link"/>
+      <child link="${side}_wheel_link"/>
+      <origin xyz="${pos_x} ${pos_y} ${pos_z}" rpy="0 0 0"/>
+      <command_interface name="velocity" />
+      <state_interface name="position" />
+      <state_interface name="velocity" />
+    </joint>
     </xacro:macro>
 </robot>

File: minibot_description/urdf/minibot_ros2_control.urdf.xacro (robot description, xacro)
@@ -15,5 +15,5 @@
                 </hardware>
             </xacro:unless>
-            <joint name="fl_wheel_joint">
+            <!-- <joint name="fl_wheel_joint">
                 <command_interface name="velocity" />
                 <state_interface name="position" />
@@ -34,8 +34,8 @@
                 <state_interface name="position" />
                 <state_interface name="velocity" />
-            </joint>
+            </joint> -->
             <gpio name="gpio">
-                <!-- <command_interface name="set_enable_motor"/>
-                <state_interface name="motor_enabled"/> -->
+                <command_interface name="set_enable_motor"/>
+                <state_interface name="motor_enabled"/>
                 <command_interface name="set_l_lamp_command"/>
                 <command_interface name="set_r_lamp_command"/>

File: minibot_description/urdf/robot.urdf.xacro (robot description, xacro)
@@ -1,5 +1,6 @@
 <?xml version="1.0"?>
 <robot xmlns:xacro="http://ros.org/wiki/xacro" name="aidl200">
-    <xacro:include filename="$(find minibot_description)/urdf/common/inertia_macro.urdf.xacro"/>
+    <xacro:include filename="$(find minibot_description)/urdf/mecanum_properties.urdf.xacro"/>
+    <xacro:include filename="$(find minibot_description)/urdf/imu.urdf.xacro"/>
     <xacro:include filename="$(find minibot_description)/urdf/minibot.urdf.xacro"/>
     <xacro:include filename="$(find minibot_description)/urdf/minibot_gazebo.urdf.xacro"/>
@@ -8,12 +9,57 @@
     <xacro:arg name="is_sim" default="false"/>
     <xacro:arg name="robot_port_name" default="/dev/ttySTM32"/>
-    <xacro:arg name="robot_baudrate" default="500000"/>
+    <xacro:arg name="robot_baudrate" default="1000000"/>
     <xacro:property name="prefix" value="$(arg prefix)"/>
     <!-- insert robot base -->
-    <xacro:insert_robot prefix="$(arg prefix)"/>
+    <xacro:insert_robot
+        prefix="$(arg prefix)"
+        length="${base_length}"
+        width="${base_width}"
+        height="${base_height}"
+        mass="${base_mass}"
+        wheel_radius="${wheel_radius}"
+        wheel_pos_z="${wheel_pos_z}"
+    />
     <xacro:insert_ros2_control prefix="$(arg prefix)" is_sim="$(arg is_sim)" robot_port_name="$(arg robot_port_name)" robot_baudrate="$(arg robot_baudrate)"/>
     <xacro:if value="$(arg is_sim)">
         <xacro:insert_gazebo prefix="$(arg prefix)"/>
     </xacro:if>
+    <xacro:mecanum_wheel
+    side="fl"
+   radius="${wheel_radius}"
+    width="${wheel_width}"
+    pos_x="${wheel_pos_x}"
+    pos_y="${wheel_pos_y}"
+    pos_z="${wheel_pos_z}"
+    mass="${wheel_mass}"
+  />
+  <xacro:mecanum_wheel
+    side="fr"
+    radius="${wheel_radius}"
+    width="${wheel_width}"
+    pos_x="${wheel_pos_x}"
+    pos_y="${-wheel_pos_y}"
+    pos_z="${wheel_pos_z}"
+    mass="${wheel_mass}"
+  />
+  <xacro:mecanum_wheel
+    side="rl"
+    radius="${wheel_radius}"
+    width="${wheel_width}"
+    pos_x="${-wheel_pos_x}"
+    pos_y="${wheel_pos_y}"
+    pos_z="${wheel_pos_z}"
+    mass="${wheel_mass}"
+  />
+  <xacro:mecanum_wheel
+    side="rr"
+    radius="${wheel_radius}"
+    width="${wheel_width}"
+    pos_x="${-wheel_pos_x}"
+    pos_y="${-wheel_pos_y}"
+    pos_z="${wheel_pos_z}"
+    mass="${wheel_mass}"
+  />
+  <xacro:imu/>
     <!-- insert ydlidar_x2 lidar -->
     <link name="${prefix}ydlidar_lidar_mount">
