Commit message: ros2 control add mecanum

File: minibot_description/urdf/minibot_ros2_control.urdf.xacro (robot description, xacro)
@@ -15,23 +15,27 @@
                 </hardware>
             </xacro:unless>
-            <joint name="${prefix}l_wheel_joint">
-                <command_interface name="velocity">
-                    <param name="min">-1.0</param>
-                    <param name="max">1.0</param>
-                </command_interface>
-                <state_interface name="position"/>
-                <state_interface name="velocity"/>
+            <joint name="fl_wheel_joint">
+                <command_interface name="velocity" />
+                <state_interface name="position" />
+                <state_interface name="velocity" />
             </joint>
-            <joint name="${prefix}r_wheel_joint">
-                <command_interface name="velocity">
-                    <param name="min">-1.0</param>
-                    <param name="max">1.0</param>
-                </command_interface>
-                <state_interface name="position"/>
-                <state_interface name="velocity"/>
+            <joint name="fr_wheel_joint">
+                <command_interface name="velocity" />
+                <state_interface name="position" />
+                <state_interface name="velocity" />
+            </joint>
+            <joint name="rl_wheel_joint">
+                <command_interface name="velocity" />
+                <state_interface name="position" />
+                <state_interface name="velocity" />
+            </joint>
+            <joint name="rr_wheel_joint">
+                <command_interface name="velocity" />
+                <state_interface name="position" />
+                <state_interface name="velocity" />
             </joint>
             <gpio name="gpio">
-                <command_interface name="set_enable_motor"/>
-                <state_interface name="motor_enabled"/>
+                <!-- <command_interface name="set_enable_motor"/>
+                <state_interface name="motor_enabled"/> -->
                 <command_interface name="set_l_lamp_command"/>
                 <command_interface name="set_r_lamp_command"/>

Commit message: system update

File: minibot_description/urdf/minibot_ros2_control.urdf.xacro (robot description, xacro)
@@ -15,5 +15,5 @@
                 </hardware>
             </xacro:unless>
-            <!-- <joint name="fl_wheel_joint">
+            <joint name="fl_wheel_joint">
                 <command_interface name="velocity" />
                 <state_interface name="position" />
@@ -34,5 +34,5 @@
                 <state_interface name="position" />
                 <state_interface name="velocity" />
-            </joint> -->
+            </joint>
             <gpio name="gpio">
                 <command_interface name="set_enable_motor"/>

Commit message: change mecanum drive controller, control xacro

File: minibot_description/urdf/minibot_ros2_control.urdf.xacro (robot description, xacro)
@@ -15,20 +15,20 @@
                 </hardware>
             </xacro:unless>
-            <joint name="fl_wheel_joint">
+            <joint name="${prefix}fl_wheel_joint">
                 <command_interface name="velocity" />
                 <state_interface name="position" />
                 <state_interface name="velocity" />
             </joint>
-            <joint name="fr_wheel_joint">
+            <joint name="${prefix}fr_wheel_joint">
                 <command_interface name="velocity" />
                 <state_interface name="position" />
                 <state_interface name="velocity" />
             </joint>
-            <joint name="rl_wheel_joint">
+            <joint name="${prefix}rl_wheel_joint">
                 <command_interface name="velocity" />
                 <state_interface name="position" />
                 <state_interface name="velocity" />
             </joint>
-            <joint name="rr_wheel_joint">
+            <joint name="${prefix}rr_wheel_joint">
                 <command_interface name="velocity" />
                 <state_interface name="position" />
