Commit message: test diff drive controller

File: minibot_description/urdf/minibot_ros2_control_test.urdf.xacro (robot description, xacro)
@@ -15,23 +15,19 @@
                 </hardware>
             </xacro:unless>
-            <joint name="fl_wheel_joint">
-                <command_interface name="velocity" />
-                <state_interface name="position" />
-                <state_interface name="velocity" />
+            <joint name="${prefix}l_wheel_joint">
+                <command_interface name="velocity">
+                    <param name="min">-1.0</param>
+                    <param name="max">1.0</param>
+                </command_interface>
+                <state_interface name="position"/>
+                <state_interface name="velocity"/>
             </joint>
-            <joint name="fr_wheel_joint">
-                <command_interface name="velocity" />
-                <state_interface name="position" />
-                <state_interface name="velocity" />
-            </joint>
-            <joint name="rl_wheel_joint">
-                <command_interface name="velocity" />
-                <state_interface name="position" />
-                <state_interface name="velocity" />
-            </joint>
-            <joint name="rr_wheel_joint">
-                <command_interface name="velocity" />
-                <state_interface name="position" />
-                <state_interface name="velocity" />
+            <joint name="${prefix}r_wheel_joint">
+                <command_interface name="velocity">
+                    <param name="min">-1.0</param>
+                    <param name="max">1.0</param>
+                </command_interface>
+                <state_interface name="position"/>
+                <state_interface name="velocity"/>
             </joint>
             <gpio name="gpio">
